File: Hardware/Schematics/Gamepad/Gamepad.kicad_sch (KiCad schematic)
At the start: 32 parts, among them J1 Cable connector, J2 Controller Plug

Commit message: Mouse capacitors measured
Other:
- moved on the sheet: JJ_2, JK_2, LTRIG_1, LTRIG_2, RTRIG_1, RTRIG_2
