File: Hardware/Schematics/Audio-Path/Audio-Path.kicad_sch (KiCad schematic)
At the start: 52 parts, among them IC252 BA15218, IC253 BA15218, J501B L, J501C R_SW

Commit message: Fix audio resistor references, recommend bridging to fix level
Parts:
- renumbered R509 to R508, R508 to R509
Changed lines of the file:
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@@
   (symbol (lib_id "Device:R") (at 168.91 66.04 90) (unit 1)
     (in_bom yes) (on_board yes) (dnp no) (fields_autoplaced)
-    (property "Reference" "R509" (at 168.91 60.96 90)
+    (property "Reference" "R508" (at 168.91 60.96 90)
       (effects (font (size 1.27 1.27)))
     )
@@
       (project "Audio-Path"
         (path "/3962d1b5-09a1-4ff8-b83f-a989027d8058"
-          (reference "R509") (unit 1)
+          (reference "R508") (unit 1)
         )
       )
@@
   (symbol (lib_id "Device:R") (at 172.72 72.39 180) (unit 1)
     (in_bom yes) (on_board yes) (dnp no)
-    (property "Reference" "R508" (at 173.99 71.12 0)
+    (property "Reference" "R509" (at 173.99 71.12 0)
       (effects (font (size 1.27 1.27)) (justify right))
     )
@@
       (project "Audio-Path"
         (path "/3962d1b5-09a1-4ff8-b83f-a989027d8058"
-          (reference "R508") (unit 1)
-        )
-      )
+          (reference "R509") (unit 1)
+        )
+      )
