File: Hardware/ControllerConn/Flex-Contact/Flex-Contact.kicad_pcb (KiCad board)
At the start: 2 copper layers, 76 x 45 mm, 6 parts

Commit message: Update hardware stuff
Other:
- board text removed: "JLCJLCJLCJLC"
Changed lines of the file:
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@@
       (layer "F.SilkS" (type "Top Silk Screen"))
       (layer "F.Paste" (type "Top Solder Paste"))
-      (layer "F.Mask" (type "Top Solder Mask") (color "#CC660080") (thickness 0.01))
+      (layer "F.Mask" (type "Top Solder Mask") (color "#C0600080") (thickness 0.01))
       (layer "F.Cu" (type "copper") (thickness 0.035))
-      (layer "dielectric 1" (type "core") (color "Polyimide") (thickness 0.02) (material "Polyimide") (epsilon_r 3.2) (loss_tangent 0.004))
+      (layer "dielectric 1" (type "core") (color "#C0600060") (thickness 0.02) (material "Polyimide") (epsilon_r 3.2) (loss_tangent 0.004))
       (layer "B.Cu" (type "copper") (thickness 0.035))
-      (layer "B.Mask" (type "Bottom Solder Mask") (color "#CC660080") (thickness 0.01))
+      (layer "B.Mask" (type "Bottom Solder Mask") (color "#C0600080") (thickness 0.01))
       (layer "B.Paste" (type "Bottom Solder Paste"))
       (layer "B.SilkS" (type "Bottom Silk Screen"))
@@
     (effects (font (size 1.5 1.4) (thickness 0.175)) (justify bottom))
   )
-  (gr_text "JLCJLCJLCJLC" (at 51 56.6) (layer "F.SilkS")
-    (effects (font (size 1 1) (thickness 0.15)))
-  )
 )
